File: flight_controller.kicad_sch (KiCad schematic)
At the start: 67 parts, among them IC1 BQ25883, IC2 STM32F722RET6, J1 Screw_Terminal_01x02, J3 USB-C, J4 MicroSD Socket, U1 BMP581, U2 TPS630702RNMR

Commit message: stm32
Parts:
- removed C23, C24, C25, C26, C31: 100nF, symbol Device:C
- removed C27, C28, C29, C32: 1μF, symbol Device:C
- removed C30: 10μF, symbol Device:C
- removed FB1: FerriteBead, symbol Device:FerriteBead
- C11, C12, C13, C15: value 22μF -> 10 μF
- C14: value 100nF -> 100 μF
- C16: value 100nF -> 10 μF
- C19, C20, C21, C22: value 100nF -> 100μF
Connections:
- net +3.3V: no longer IC2.1 (VBAT), IC2.19 (VDD_1), IC2.32 (VDD_2), IC2.48 (VDD_3), IC2.64 (VDD_4)
- net GND: no longer IC2.12 (VSSA), IC2.18 (VSS_1), IC2.31 (VSS_2), IC2.47 (VSS_3), IC2.63 (VSS_4)
Other:
- moved on the sheet: C10, C11, C12, C13, C21, C22, D1, IC2
