File: hardware/_autosave-flight_controller.kicad_pcb (KiCad board)
At the start: 2 copper layers, 50 x 50 mm, 85 parts, among them IC2 STM32F722RET6, IC3 W25Q128JVSIQ, J1 Conn_01x06, J2 Conn_01x08, J4 Conn_01x04, J5 Conn_01x04, J6 USB4105-GF-A-060, Q1 TPRT9013-33GB, SW2 SW_SPST, U1 BMP581, U2 MP9943GQ-Z, U3 USBLC6-2P6, U4 MP9943GQ-Z, Y1 Q13FC13500004, Y2 X322525MOB4SI

Commit message: layout
Parts:
- moved R14 12.5 mm to (190.5, 114.8)
- moved R15 12.5 mm to (190.5, 109.2)
- moved J6 12.0 mm to (196.7, 111.5)
- moved IC3 11.9 mm to (181.5, 115.5)
- moved C24 11.4 mm to (172.7, 46.0)
- moved C23 11.4 mm to (172.7, 43.2)
- moved C34 11.4 mm to (175.5, 43.2)
- moved FB1 9.95 mm to (182.9, 95.1), turned to 45 degrees
- moved Y2 8.36 mm to (186.6, 96.2), turned to 45 degrees
- moved Y1 7.25 mm to (189.6, 99.4), turned to 45 degrees
- moved SW2 3.64 mm to (168.5, 91.0)
- moved C5 3.50 mm to (154.2, 102.1)
- moved C1 3.44 mm to (161.7, 99.3)
- moved C2 3.44 mm to (161.7, 101.6)
- moved C3 3.44 mm to (161.7, 103.8)
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