File: hardware/_autosave-flight_controller.kicad_pcb (KiCad board)
At the start: 6 copper layers, 50 x 50 mm, 83 parts, among them IC2 STM32F722RET6, IC3 W25Q128JVSIQ, J2 Conn_01x08, J3 Conn_01x04, J4 Conn_01x04, J5 Conn_01x04, J6 USB4105-GF-A-060, Q1 TPRT9013-33GB, SW2 SW_SPST, U1 BMP581, U2 MP9943GQ-Z, U3 USBLC6-2P6, U4 MP9943GQ-Z, Y1 Q13FC13500004, Y2 X322525MOB4SI

Commit message: layout
Parts:
- moved R15 1.10 mm to (190.6, 110.3), turned to -90 degrees
Changed lines of the file:
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@@
 	(footprint "Resistor_SMD:R_01005_0402Metric"
 		(layer "F.Cu")
-		(at 190.5 109.175 90)
+		(at 190.6 110.275 -90)
 		(descr "Resistor SMD 01005 (0402 Metric), square (rectangular) end terminal, IPC-7351 nominal, (Body size source: http://www.vishay.com/docs/20056/crcw01005e3.pdf), generated with kicad-footprint-generator")
 		(tags "resistor")
@@
 		)
 		(pad "" smd roundrect
-			(at -0.275 0 90)
+			(at -0.275 0 270)
 			(size 0.27 0.27)
 			(layers "F.Paste")
@@
 		)
 		(pad "" smd roundrect
-			(at 0.275 0 90)
+			(at 0.275 0 270)
 			(size 0.27 0.27)
 			(layers "F.Paste")
@@
 		)
 		(pad "1" smd roundrect
-			(at -0.25 0 90)
+			(at -0.25 0 270)
 			(size 0.4 0.3)
 			(layers "F.Cu" "F.Mask")
@@
 		)
 		(pad "2" smd roundrect
-			(at 0.25 0 90)
+			(at 0.25 0 270)
 			(size 0.4 0.3)
 			(layers "F.Cu" "F.Mask")
@@
 	)
 	(segment
-		(start 189.301242 108.31373)
-		(end 189.001242 108.61373)
+		(start 191.1 109.1)
+		(end 191.9075 109.1)
 		(width 0.2)
 		(layer "F.Cu")
@@
 	)
 	(segment
-		(start 191.9075 109.1)
-		(end 191.408824 109.1)
+		(start 189.001242 108.61373)
+		(end 190.61373 108.61373)
 		(width 0.2)
 		(layer "F.Cu")
@@
 	)
 	(segment
-		(start 191.408824 109.1)
-		(end 190.622554 108.31373)
-		(width 0.2)
-		(layer "F.Cu")
-		(net 12)
-	)
-	(segment
-		(start 190.622554 108.31373)
-		(end 189.301242 108.31373)
+		(start 190.61373 108.61373)
+		(end 191.1 109.1)
 		(width 0.2)
 		(layer "F.Cu")
@@
 	)
 	(segment
-		(start 190.825 109.75)
-		(end 190.5 109.425)
-		(width 0.2)
+		(start 190.849 109.776)
+		(end 191.8815 109.776)
+		(width 0.15)
 		(layer "F.Cu")
 		(net 85)
 	)
 	(segment
-		(start 191.9075 109.75)
-		(end 190.825 109.75)
-		(width 0.2)
+		(start 190.6 110.025)
+		(end 190.849 109.776)
+		(width 0.15)
 		(layer "F.Cu")
 		(net 85)
@@
 		(priority 1)
 		(connect_pads
-			(clearance 0.3)
+			(clearance 0.2)
 		)
 		(min_thickness 0.25)
