File: hardware/flight_controller.kicad_sch (KiCad schematic)
At the start: 67 parts, among them IC1 BQ25883, IC2 STM32F722RET6, J1 Screw_Terminal_01x02, J3 USB-C, J4 MicroSD Socket, U1 BMP581, U2 TPS630702RNMR

Commit message: stm32
Parts:
- added C33, C34: 6.8pF, symbol Device:C
- added C35, C36: 20pF, symbol Device:C
- added C37: 100nF, symbol Device:C
- added R22: 5.23KΩ, symbol Device:R
- added SW1, SW2: SW_SPST, symbol Switch:SW_SPST
- added Y1: Q13FC13500004, drone_footprints:Q13FC13500004, symbol drone_symbols:Q13FC13500004
- added Y2: X322525MOB4SI, drone_footprints:X322525MOB4SI, symbol drone_symbols:X322525MOB4SI
Connections:
- net +3.3V: now also SW2.1 (A)
- net GND: now also C33.1, C34.1, C35.1, C36.1, C37.2, R22.1, SW1.1 (A), Y2.3 (CRYSTAL__2), Y2.4 (GND_2)
- net LSE_IN: now reaches IC2.3 (PC14-OSC32_IN)
- net LSE_IN: now also C33.2, Y1.1
- net LSE_OUT: now reaches IC2.4 (PC15-OSC32_OUT)
- net LSE_OUT: now also C34.2, Y1.2
- net HSE_IN: now reaches IC2.5 (PH0-OSC_IN)
- net HSE_IN: now also C35.2, Y2.1 (CRYSTAL__1)
- net HSE_OUT: now reaches IC2.6 (PH1-OSC_OUT)
- net HSE_OUT: now also C36.2, Y2.2 (GND_1)
- new net BOOT: R22.2, SW2.2 (B)
- new net RESET: C37.1, SW1.2 (B)
Other:
- moved on the sheet: C23, C24, C25, C26, C27, C28, C29, C30, C31, C32, FB1, IC2

Commit message: changed components
Parts:
- removed C1: 1μF, symbol Device:C
- removed C10, C2, C5, C7, C8, C9: 10 μF, symbol Device:C
- removed C11, C12, C13: 22μF, symbol Device:C
- removed C14: 100nF, symbol Device:C
- removed C3: 4.7 μF, symbol Device:C
- removed C4: 47 μF, symbol Device:C
- removed C6: 44μF, symbol Device:C
- removed D2: LED, symbol Device:LED
- removed IC1: BQ25883, drone_footprints:QFN50P400X400X100-25N-D, symbol drone_symbols:BQ25883RGER
- removed J1: Screw_Terminal_01x02, symbol Connector:Screw_Terminal_01x02
- removed J4: MicroSD Socket, drone_footprints:MicroSD_socket, symbol drone_symbols:GTFP08441BEU
- removed L1: 1μH, symbol Device:L
- removed L2: 1 μH, symbol Device:L
- removed R10: 30.1KΩ, symbol Device:R
- removed R11, R12, R18, R19, R20, R21, R3, R4, R5, R6, R7: 10KΩ, symbol Device:R
- removed R13: 100KΩ, symbol Device:R
- removed R8: 383Ω, symbol Device:R
- removed R9: 5.23KΩ, symbol Device:R
- removed U2: TPS630702RNMR, drone_footprints:VREG_TPS630702RNMR, symbol drone_symbols:TPS630702RNMR
- added IC3: W25Q128JVSIQ, drone_footprints:SOIC127P790X216-8N, symbol drone_symbols:W25Q128JVSIQ
- added U2: MP9943GQ-Z, drone_footprints:QFN-8_MP9943_MNP, symbol drone_symbols:MP9943GQ-Z
- R16, R17: value 10KΩ -> 10k
Connections:
- net SD_DAT3 is gone; now on net +3.3v: R17.1
- net +3.3V: no longer R16.2, R17.2
- net GND: no longer C15.2, C17.2, C18.2, C19.2, C20.2, C21.2, C22.2, C23.1, C24.1, C25.1, C26.1, C27.1, C28.1, C29.1, C30.1, C31.1, C32.1, C33.1, C34.1, C35.1, C36.1, C37.2, D1.6 (GND), IC2.12 (VSSA), IC2.18 (VSS_1), IC2.31 (VSS_2), IC2.47 (VSS_3), IC2.63 (VSS_4), PS1.1 (GND), R15.1, R22.1, SW1.1 (A), U1.3 (VSS_1), U1.5 (SDO), U1.6 (CSB), U1.8 (VSS_2), U1.9 (VSS_3), Y2.3 (CRYSTAL__2), Y2.4 (GND_2)
- net SD_CMD renamed +3.3v
- net +3.3v: now also IC3.8 (VCC)
- net VBUS renamed VBUS_A
- new net: IC3.3 (/WP_(IO2)), R17.2
- new net: IC3.7 (/HOLD_OR_/RESET_(IO3)), R16.2
- new net CS_FLASH: IC3.1 (/CS)
- new net GNDREF: C15.2, C17.2, C18.2, C19.2, C20.2, C21.2, C22.2, C23.1, C24.1, C25.1, C26.1, C27.1, C28.1, C29.1, C30.1, C31.1, C32.1, C33.1, C34.1, C35.1, C36.1, C37.2, D1.6 (GND), IC2.12 (VSSA), IC2.18 (VSS_1), IC2.31 (VSS_2), IC2.47 (VSS_3), IC2.63 (VSS_4), IC3.4 (GND), PS1.1 (GND), R15.1, R22.1, SW1.1 (A), U1.3 (VSS_1), U1.5 (SDO), U1.6 (CSB), U1.8 (VSS_2), U1.9 (VSS_3), Y2.3 (CRYSTAL__2), Y2.4 (GND_2)
- new net SPI_MISO: IC3.2 (DO_(IO1))
- new net SPI_MOSI: IC3.5 (DI_(IO0))
- new net SPI_SCLK: IC3.6 (CLK)
- new net VBAT: U2.7 (IN)
- no-connect marks 17 -> 15
Other:
- note added: "BAROMETER"
- note added: "BUCK VOLTAGE REGULATOR (VIN: 9V-36V)"
- note added: "INERTIA MEASUREMENT UNIT"
- note added: "SPI FLASH"
- note added: "USB-C CONNECTOR"
- moved on the sheet: C21, C22, D1

Commit message: interfaces
Parts:
- removed C15, C17, C18: 22μF, symbol Device:C
- removed C16, C37: 100nF, symbol Device:C
- removed L3: 6.8μH, symbol Device:L
- removed PS1: LMR51430, drone_footprints:LMR51430, symbol drone_symbols:LMR51430XDDCR
- removed R14: 100KΩ, symbol Device:R
- removed R15: 22.1KΩ, symbol Device:R
- removed SW1: SW_SPST, symbol Switch:SW_SPST
- added C1, C2, C3: 10μF, symbol Device:C
- added C4, C5: 100nF, symbol Device:C
- added C6, C7: 22μF, symbol Device:C
- added C8, C9: 1μF, symbol Device:C
- added D2: BAT54C, Package_TO_SOT_SMD:SOT-23, symbol Diode:BAT54C
- added D3, D4, D5: 1N4148WT, Diode_SMD:D_SOD-523, symbol Diode:1N4148WT
- added J1: Conn_01x06, symbol Connector_Generic:Conn_01x06
- added J2: Conn_01x08, symbol Connector_Generic:Conn_01x08
- added L1: 10μH, symbol Device:L
- added Q1: TPRT9013-33GB, drone_footprints:SOT95P280X125-5N, symbol drone_symbols:TPRT9013-33GB
- added R10, R9: 22Ω, symbol Device:R
- added R11: 150Ω, symbol Device:R
- added R12: 300Ω, symbol Device:R
- added R13: 470Ω, symbol Device:R
- added R3, R4: 100KΩ, symbol Device:R
- added R5: 20Ω, symbol Device:R
- added R6: 51KΩ, symbol Device:R
- added R7: 41.2KΩ, symbol Device:R
- added R8: 7.5KΩ, symbol Device:R
- added U3: USBLC6-2P6, Package_TO_SOT_SMD:SOT-666, symbol Power_Protection:USBLC6-2P6
- R1: value R1 5.1K -> R1 5.1KΩ
- R2: value R2 5.1K -> R2 5.1KΩ
Connections:
- net +3.3V: now also C8.1, Q1.5 (VOUT)
- net GNDREF: now also U2.5 (GND), C1.2, C2.2, C3.2, C4.2, C6.2, C7.2, C8.2, C9.2, J1.2 (Pin_2), J1.5 (Pin_5), J2.2 (Pin_2), Q1.2 (GND), R11.1, R12.1, R13.1, R8.1, U3.2 (GND)
- net USB_DN: now also R9.2, U3.1 (I/O1)
- net USB_DP: now also R10.2, U3.3 (I/O2)
- net VBAT: now also C1.1, C2.1, C3.1, J1.1 (Pin_1), J2.1 (Pin_1), R4.1
- net at U2.1 (FB): now also R6.1
- net at U2.2 (VCC): now also C4.1, R3.2
- net at U2.3 (EN/SYNC): now also R4.2
- net at U2.4 (BST): now also R5.1
- net at U2.6 (SW): now also C5.1, L1.1
- net at U2.8 (PG): now also R3.1
- new net: R6.2, R7.1, R8.2
- new net: D5.1 (K), R13.2
- new net: C5.2, R5.2
- new net: R10.1, U3.4 (I/O2)
- new net: R9.1, U3.6 (I/O1)
- new net: D4.1 (K), R12.2
- new net: D3.1 (K), R11.2
- new net +3V: D3.2 (A)
- new net +5V: C6.1, C7.1, C9.1, D2.3, D4.2 (A), L1.2, Q1.1 (VIN), Q1.3 (CE), R7.2, U3.5 (VBUS)
- new net +5VBAT: D2.2
- new net +5VUSB: D2.1
- new net ANALOG_PIN: J2.3 (Pin_3)
- new net STATUS: D5.2 (A)
- new net TIM2_CH1: J2.4 (Pin_4)
- new net TIM2_CH2: J2.5 (Pin_5)
- new net TIM2_CH3: J2.6 (Pin_6)
- new net TIM2_CH4: J2.7 (Pin_7)
- new net UART4_RX: J2.8 (Pin_8)
- new net UART_RX: J1.3 (Pin_3)
- new net UART_TX: J1.4 (Pin_4)
- no-connect marks 15 -> 16
Other:
- note added: "3.3 LDO"
- note added: "BOOT SWITCH"
- note added: "CRYSTALS"
- note added: "DECOUPLING"
- note added: "ESC"
- note added: "LEDS"
- note added: "POWER DIODE"
- note added: "STM 32"
- note added: "USB DIODE"
- note added: "VTX"
- moved on the sheet: C23, C24, C25, C26, C27, C28, C29, C30, C31, C32, C33, C34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

Commit message: stm32 interfaces
Parts:
- added J4, J5: Conn_01x04, symbol Connector_Generic:Conn_01x04
Connections:
- net SPI_MISO is gone; now on net SPI1_MISO: IC3.2 (DO_(IO1))
- net SPI_MOSI is gone; now on net SPI1_MOSI: IC3.5 (DI_(IO0))
- net SPI_SCLK is gone; now on net SPI1_SCLK: IC3.6 (CLK)
- net UART_TX is gone; now on net USART6_TX: J1.4 (Pin_4)
- net +5V: now also J4.1 (Pin_1), J5.1 (Pin_1)
- net ANALOG_PIN: now also IC2.22 (PA6)
- net BMP_INT: now also IC2.59 (PB7)
- net BMP_SCK: now also IC2.61 (PB8)
- net BMP_SDI: now also IC2.62 (PB9)
- net BOOT: now also IC2.60 (BOOT0)
- net CS_FLASH: now also IC2.50 (PA15)
- net GNDREF: now also J4.4 (Pin_4), J5.4 (Pin_4)
- net ICM_CS: now also IC2.33 (PB12)
- net ICM_INT2: now also IC2.25 (PB0); no longer D1.4 (INT1/INT)
- net ICM_SCLK: now also IC2.34 (PB13)
- net ICM_SDI: now also IC2.10 (PC2); no longer D1.1 (AP_SDO/AP_AD0)
- net STATUS: now also IC2.41 (PA8)
- net TIM2_CH1: now also IC2.14 (PA0-WKUP)
- net TIM2_CH2: now also IC2.15 (PA1)
- net TIM2_CH3: now also IC2.28 (PB10)
- net TIM2_CH4: now also IC2.29 (PB11)
- net USB_DN: now also IC2.44 (PA11)
- net USB_DP: now also IC2.45 (PA12)
- net USART2_TX: now reaches IC2.16 (PA2)
- net USART2_RX: now reaches IC2.17 (PA3)
- net SPI1_SCLK: now reaches IC2.21 (PA5)
- net SPI1_MOSI: now reaches IC2.23 (PA7)
- net ICM_INT1: now reaches IC2.24 (PC4)
- net ICM_INT1: now also D1.4 (INT1/INT)
- net USART6_TX: now reaches IC2.37 (PC6)
- net USART6_RX: now reaches IC2.38 (PC7)
- net USART1_TX: now reaches IC2.42 (PA9)
- net USART1_TX: now also J4.3 (Pin_3)
- net USART1_RX: now reaches IC2.43 (PA10)
- net USART1_RX: now also J4.2 (Pin_2)
- net USART5_TX: now reaches IC2.53 (PC12)
- net USART5_TX: now also J5.3 (Pin_3)
- net USART5_RX: now reaches IC2.54 (PD2)
- net USART5_RX: now also J5.2 (Pin_2)
- net SPI1_MISO: now reaches IC2.56 (PB4)
- net ICM_SDO: now reaches IC2.9 (PC1)
- net ICM_SDO: now also D1.1 (AP_SDO/AP_AD0)
- net UART4_RX renamed UART2_RX
- net UART_RX renamed UASRT6_RX
Other:
- note added: "GPS"
- note added: "RADIO TRANSCIEVER"
- moved on the sheet: C32, FB1, IC2

Commit message: footprints
Parts:
- C1, C2, C3, C30, C6, C7: footprint (none) -> Capacitor_SMD:C_0805_2012Metric
- C19, C20, C21, C22, C23, C24, C25, C26, C31, C33, C34, C35, C36, C4, C5: footprint (none) -> Capacitor_SMD:C_0402_1005Metric
- C27, C28, C29, C32, C8, C9: footprint (none) -> Capacitor_SMD:C_0201_0603Metric
- D1: footprint QFN50P300X250X78-14N -> drone_footprints:QFN50P300X250X78-14N
- FB1: footprint (none) -> Inductor_SMD:L_0603_1608Metric
- J1: footprint (none) -> Connector_PinHeader_2.54mm:PinHeader_1x06_P2.54mm_Vertical
- J2: footprint (none) -> Connector_JST:JST_SH_SM08B-SRSS-TB_1x08-1MP_P1.00mm_Horizontal
- J4, J5: footprint (none) -> Connector_PinHeader_2.54mm:PinHeader_1x04_P2.54mm_Vertical
- L1, SW2: footprint (none) -> Button_Switch_SMD:SW_Push_1P1T-SH_NO_CK_KMR2xxG
- R1, R10, R11, R12, R13, R16, R17, R2, R22, R3, R4, R5, R6, R7, R8, R9: footprint (none) -> Resistor_SMD:R_0603_1608Metric
Changed lines of the file:
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@@
 			)
 		)
-		(property "Footprint" ""
+		(property "Footprint" "Resistor_SMD:R_0603_1608Metric"
 			(at 95.25 140.208 90)
 			(effects
@@
 			)
 		)
-		(property "Footprint" ""
+		(property "Footprint" "Resistor_SMD:R_0603_1608Metric"
 			(at 53.34 140.208 90)
 			(effects
@@
 			)
 		)
-		(property "Footprint" ""
+		(property "Footprint" "Button_Switch_SMD:SW_Push_1P1T-SH_NO_CK_KMR2xxG"
 			(at 284.48 194.31 0)
 			(effects
@@
 			)
 		)
-		(property "Footprint" ""
+		(property "Footprint" "Capacitor_SMD:C_0402_1005Metric"
 			(at 345.7448 229.87 0)
 			(effects
@@
 			)
 		)
-		(property "Footprint" ""
+		(property "Footprint" "Resistor_SMD:R_0603_1608Metric"
 			(at 27.94 109.728 90)
 			(effects
@@
 			)
 		)
-		(property "Footprint" ""
+		(property "Footprint" "Capacitor_SMD:C_0402_1005Metric"
 			(at 343.2048 205.74 0)
 			(effects
@@
 			)
 		)
-		(property "Footprint" ""
+		(property "Footprint" "Capacitor_SMD:C_0402_1005Metric"
 			(at 97.4852 182.88 0)
 			(effects
@@
 			)
 		)
-		(property "Footprint" ""
+		(property "Footprint" "Inductor_SMD:L_0603_1608Metric"
 			(at 234.95 121.158 90)
 			(effects
@@
 			)
 		)
-		(property "Footprint" ""
+		(property "Footprint" "Resistor_SMD:R_0603_1608Metric"
 			(at 312.928 241.3 90)
 			(effects
@@
 			)
 		)
-		(property "Footprint" ""
+		(property "Footprint" "Capacitor_SMD:C_0402_1005Metric"
 			(at 373.6848 229.87 0)
 			(effects
@@
 			)
 		)
-		(property "Footprint" ""
+		(property "Footprint" "Capacitor_SMD:C_0805_2012Metric"
 			(at 211.1248 86.36 0)
 			(effects
@@
 			)
 		)
-		(property "Footprint" ""
+		(property "Footprint" "Capacitor_SMD:C_0201_0603Metric"
 			(at 203.5048 86.36 0)
 			(effects
@@
 			)
 		)
-		(property "Footprint" ""
+		(property "Footprint" "Button_Switch_SMD:SW_Push_1P1T-SH_NO_CK_KMR2xxG"
 			(at 110.49 107.95 0)
 			(effects
@@
 			)
 		)
-		(property "Footprint" ""
+		(property "Footprint" "Capacitor_SMD:C_0402_1005Metric"
 			(at 173.0248 86.36 0)
 			(effects
@@
 			)
 		)
-		(property "Footprint" ""
+		(property "Footprint" "Capacitor_SMD:C_0402_1005Metric"
 			(at 253.6952 257.81 0)
 			(effects
@@
 			)
 		)
-		(property "Footprint" ""
+		(property "Footprint" "Capacitor_SMD:C_0402_1005Metric"
 			(at 166.6748 86.36 0)
 			(effects
@@
 			)
 		)
-		(property "Footprint" ""
+		(property "Footprint" "Capacitor_SMD:C_0402_1005Metric"
 			(at 143.8148 86.36 0)
 			(effects
@@
 			)
 		)
-		(property "Footprint" ""
+		(property "Footprint" "Resistor_SMD:R_0603_1608Metric"
 			(at 53.34 132.588 90)
 			(effects
@@
 			)
 		)
-		(property "Footprint" ""
+		(property "Footprint" "Capacitor_SMD:C_0805_2012Metric"
 			(at 126.6952 115.57 0)
 			(effects
@@
 			)
 		)
-		(property "Footprint" ""
+		(property "Footprint" "Capacitor_SMD:C_0805_2012Metric"
 			(at 106.3752 88.9 0)
 			(effects
@@
 			)
 		)
-		(property "Footprint" ""
+		(property "Footprint" "Connector_PinHeader_2.54mm:PinHeader_1x04_P2.54mm_Vertical"
 			(at 203.2 151.13 0)
 			(effects
@@
 			)
 		)
-		(property "Footprint" ""
+		(property "Footprint" "Connector_JST:JST_SH_SM08B-SRSS-TB_1x08-1MP_P1.00mm_Horizontal"
 			(at 213.36 121.92 0)
 			(effects
@@
 			)
 		)
-		(property "Footprint" ""
+		(property "Footprint" "Capacitor_SMD:C_0402_1005Metric"
 			(at 159.0548 86.36 0)
 			(effects
@@
 			)
 		)
-		(property "Footprint" ""
+		(property "Footprint" "Capacitor_SMD:C_0805_2012Metric"
 			(at 113.9952 88.9 0)
 			(effects
@@
 			)
 		)
-		(property "Footprint" ""
+		(property "Footprint" "Resistor_SMD:R_0603_1608Metric"
 			(at 294.64 36.068 90)
 			(effects
@@
 			)
 		)
-		(property "Footprint" ""
+		(property "Footprint" "Connector_PinHeader_2.54mm:PinHeader_1x04_P2.54mm_Vertical"
 			(at 355.6 33.02 0)
 			(effects
@@
 			)
 		)
-		(property "Footprint" ""
+		(property "Footprint" "Capacitor_SMD:C_0201_0603Metric"
 			(at 188.2648 86.36 0)
 			(effects
@@
 			)
 		)
-		(property "Footprint" ""
+		(property "Footprint" "Resistor_SMD:R_0603_1608Metric"
 			(at 295.148 241.3 90)
 			(effects
@@
 			)
 		)
-		(property "Footprint" ""
+		(property "Footprint" "Capacitor_SMD:C_0402_1005Metric"
 			(at 16.2052 119.38 0)
 			(effects
@@
 			)
 		)
-		(property "Footprint" "QFN50P300X250X78-14N"
+		(property "Footprint" "drone_footprints:QFN50P300X250X78-14N"
 			(at 229.87 307.01 0)
 			(effects
@@
 			)
 		)
-		(property "Footprint" ""
+		(property "Footprint" "Capacitor_SMD:C_0402_1005Metric"
 			(at 101.2952 124.46 0)
 			(effects
@@
 			)
 		)
-		(property "Footprint" ""
+		(property "Footprint" "Capacitor_SMD:C_0201_0603Metric"
 			(at 122.8852 45.72 0)
 			(effects
@@
 			)
 		)
-		(property "Footprint" ""
+		(property "Footprint" "Capacitor_SMD:C_0402_1005Metric"
 			(at 69.5452 168.91 0)
 			(effects
@@
 			)
 		)
-		(property "Footprint" ""
+		(property "Footprint" "Capacitor_SMD:C_0402_1005Metric"
 			(at 187.6552 279.4 0)
 			(effects
@@
 			)
 		)
-		(property "Footprint" ""
+		(property "Footprint" "Capacitor_SMD:C_0201_0603Metric"
 			(at 195.8848 86.36 0)
 			(effects
@@
 			)
 		)
-		(property "Footprint" ""
+		(property "Footprint" "Resistor_SMD:R_0603_1608Metric"
 			(at 13.462 97.79 90)
 			(effects
@@
 			)
 		)
-		(property "Footprint" ""
+		(property "Footprint" "Resistor_SMD:R_0603_1608Metric"
 			(at 297.688 198.12 90)
 			(effects
@@
 			)
 		)
-		(property "Footprint" ""
+		(property "Footprint" "Capacitor_SMD:C_0805_2012Metric"
 			(at 98.7552 88.9 0)
 			(effects
@@
 			)
 		)
-		(property "Footprint" ""
+		(property "Footprint" "Resistor_SMD:R_0603_1608Metric"
 			(at 35.052 254 90)
 			(effects
@@
 			)
 		)
-		(property "Footprint" ""
+		(property "Footprint" "Resistor_SMD:R_0603_1608Metric"
 			(at 19.05 47.498 90)
 			(effects
@@
 			)
 		)
-		(property "Footprint" ""
+		(property "Footprint" "Resistor_SMD:R_0603_1608Metric"
 			(at 81.28 55.118 90)
 			(effects
@@
 			)
 		)
-		(property "Footprint" ""
+		(property "Footprint" "Capacitor_SMD:C_0402_1005Metric"
 			(at 151.4348 86.36 0)
 			(effects
@@
 			)
 		)
-		(property "Footprint" ""
+		(property "Footprint" "Resistor_SMD:R_0603_1608Metric"
 			(at 75.438 142.24 90)
 			(effects
@@
 			)
 		)
-		(property "Footprint" ""
+		(property "Footprint" "Resistor_SMD:R_0603_1608Metric"
 			(at 294.64 38.608 90)
 			(effects
@@
 			)
 		)
-		(property "Footprint" ""
+		(property "Footprint" "Capacitor_SMD:C_0805_2012Metric"
 			(at 119.0752 115.57 0)
 			(effects
@@
 			)
 		)
-		(property "Footprint" ""
+		(property "Footprint" "Capacitor_SMD:C_0201_0603Metric"
 			(at 317.8048 156.21 0)
 			(effects
@@
 			)
 		)
-		(property "Footprint" ""
+		(property "Footprint" "Capacitor_SMD:C_0402_1005Metric"
 			(at 395.2748 205.74 0)
 			(effects
@@
 			)
 		)
-		(property "Footprint" ""
+		(property "Footprint" "Capacitor_SMD:C_0201_0603Metric"
 			(at 168.6052 52.07 0)
 			(effects
@@
 			)
 		)
-		(property "Footprint" ""
+		(property "Footprint" "Resistor_SMD:R_0603_1608Metric"
 			(at 97.282 254 90)
 			(effects
@@
 			)
 		)
-		(property "Footprint" ""
+		(property "Footprint" "Resistor_SMD:R_0603_1608Metric"
 			(at 277.368 242.57 90)
 			(effects
@@
 			)
 		)
-		(property "Footprint" ""
+		(property "Footprint" "Connector_PinHeader_2.54mm:PinHeader_1x06_P2.54mm_Vertical"
 			(at 161.29 119.38 0)
 			(effects

Commit message: layout
Parts:
- removed J3: USB-C, drone_footprints:TE_2129691-2, symbol drone_symbols:2129691-2
- added C10, C12: 100nF, Capacitor_SMD:C_0402_1005Metric, symbol Device:C
- added C11, C13, C14: 10μF, Capacitor_SMD:C_0805_2012Metric, symbol Device:C
- added C15, C16: 22μF, Capacitor_SMD:C_0805_2012Metric, symbol Device:C
- added J6: USB4105-GF-A-060, drone_footprints:GCT_USB4105-GF-A-060, symbol drone_symbols:USB4105-GF-A-060
- added L2: 10μH, Inductor_SMD:L_2010_5025Metric, symbol Device:L
- added R14: R2 5.1KΩ, Resistor_SMD:R_01005_0402Metric, symbol Device:R
- added R15: R1 5.1KΩ, Resistor_SMD:R_01005_0402Metric, symbol Device:R
- added R18: 20Ω, Resistor_SMD:R_01005_0402Metric, symbol Device:R
- added R19: 51KΩ, Resistor_SMD:R_01005_0402Metric, symbol Device:R
- added R20: 3.92KΩ, Resistor_SMD:R_01005_0402Metric, symbol Device:R
- added R21: 41.2KΩ, Resistor_SMD:R_01005_0402Metric, symbol Device:R
- added U4: MP9943GQ-Z, drone_footprints:QFN-8_MP9943_MNP, symbol drone_symbols:MP9943GQ-Z
- J1: footprint Connector_PinHeader_2.54mm:PinHeader_1x06_P2.54mm_Vertical -> Connector_PinHeader_1.27mm:PinHeader_1x06_P1.27mm_Vertical
- J4, J5: footprint Connector_PinHeader_2.54mm:PinHeader_1x04_P2.54mm_Vertical -> Connector_PinHeader_1.27mm:PinHeader_1x04_P1.27mm_Vertical
- L1: footprint Button_Switch_SMD:SW_Push_1P1T-SH_NO_CK_KMR2xxG -> Inductor_SMD:L_2010_5025Metric
- R1: value R1 5.1KΩ -> 100KΩ; footprint Resistor_SMD:R_0603_1608Metric -> Resistor_SMD:R_01005_0402Metric
- R10, R11, R12, R13, R16, R17, R22, R3, R4, R5, R6, R7, R8, R9: footprint Resistor_SMD:R_0603_1608Metric -> Resistor_SMD:R_01005_0402Metric
- R2: value R2 5.1KΩ -> 100KΩ; footprint Resistor_SMD:R_0603_1608Metric -> Resistor_SMD:R_01005_0402Metric
Connections:
- net GND: now also J6.A1_B12 (GND), J6.B1_A12 (GND), J6.SH1 (SHELL_GND), J6.SH2 (SHELL_GND), J6.SH3 (SHELL_GND), J6.SH4 (SHELL_GND), R14.1, R15.2; no longer R1.2, R2.1
- net GNDREF: now also C10.2, C11.2, C13.2, C14.2, C15.2, C16.2, R20.1, U4.5 (GND)
- net USB_DN: now also J6.A7 (DN1), J6.B7 (DN2)
- net USB_DP: now also J6.A6 (DP1), J6.B6 (DP2)
- net VBAT: now also R2.1, C11.1, C13.1, C14.1, U4.7 (IN); no longer J1.1 (Pin_1)
- net at R1.1: now also U4.8 (PG)
- net at R2.2: now also U4.3 (EN/SYNC)
- new net: C10.1, R1.2, U4.2 (VCC)
- new net: R19.2, R20.2, R21.1
- new net: J6.A5 (CC1), R14.2
- new net: J6.B5 (CC2), R15.1
- new net: C12.1, L2.1, U4.6 (SW)
- new net: C12.2, R18.2
- new net: R19.1, U4.1 (FB)
- new net: R18.1, U4.4 (BST)
- new net +9V: C15.1, C16.1, J1.1 (Pin_1), L2.2, R21.2
- new net VBUS: J6.A4_B9 (VBUS), J6.B4_A9 (VBUS)
- no-connect marks 16 -> 8
Other:
- note added: "BUCK VOLTAGE REGULATOR VIN: 9V-36V, VOUT: 5V"
- note added: "BUCK VOLTAGE REGULATOR VIN: 9V-36V, VOUT: 9V"
- note removed: "BUCK VOLTAGE REGULATOR (VIN: 9V-36V)"
- moved on the sheet: C32, C33, C34, C35, C36, FB1, IC2, Y1, Y2

Commit message: resized board
Parts:
- J1: footprint Connector_PinHeader_1.27mm:PinHeader_1x06_P1.27mm_Vertical -> Connector_PinHeader_2.54mm:PinHeader_1x06_P2.54mm_Vertical
- J4, J5: footprint Connector_PinHeader_1.27mm:PinHeader_1x04_P1.27mm_Vertical -> Connector_PinHeader_2.54mm:PinHeader_1x04_P2.54mm_Vertical
Changed lines of the file:
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@@
 			)
 		)
-		(property "Footprint" "Connector_PinHeader_1.27mm:PinHeader_1x04_P1.27mm_Vertical"
+		(property "Footprint" "Connector_PinHeader_2.54mm:PinHeader_1x04_P2.54mm_Vertical"
 			(at 203.2 151.13 0)
 			(effects
@@
 			)
 		)
-		(property "Footprint" "Connector_PinHeader_1.27mm:PinHeader_1x04_P1.27mm_Vertical"
+		(property "Footprint" "Connector_PinHeader_2.54mm:PinHeader_1x04_P2.54mm_Vertical"
 			(at 355.6 33.02 0)
 			(effects
@@
 			)
 		)
-		(property "Footprint" "Connector_PinHeader_1.27mm:PinHeader_1x06_P1.27mm_Vertical"
+		(property "Footprint" "Connector_PinHeader_2.54mm:PinHeader_1x06_P2.54mm_Vertical"
 			(at 161.29 119.38 0)
 			(effects

Commit message: layout
Parts:
- removed J1: Conn_01x06, Connector_PinHeader_2.54mm:PinHeader_1x06_P2.54mm_Vertical, symbol Connector_Generic:Conn_01x06
- added J3: Conn_01x04, Connector_PinHeader_2.54mm:PinHeader_1x04_P2.54mm_Vertical, symbol Connector_Generic:Conn_01x04
Connections:
- net +5VUSB is gone; now on net VBUS: D2.1
- net +5V: now also J4.4 (Pin_4), J5.4 (Pin_4); no longer J4.1 (Pin_1), J5.1 (Pin_1)
- net +9V: now also J3.4 (Pin_4)
- net GNDREF: now also J4.1 (Pin_1), J5.1 (Pin_1), J3.1 (Pin_1); no longer J4.4 (Pin_4), J5.4 (Pin_4)
- net UASRT6_RX: now also J3.2 (Pin_2)
- net USART6_TX: now also J3.3 (Pin_3)
- no-connect marks 8 -> 7
