File: hardware/flight_controller.kicad_sch (KiCad schematic)
At the start: 77 parts, among them IC2 STM32F722RET6, IC3 W25Q128JVSIQ, J1 Conn_01x03, J2 Conn_01x08, J3 Conn_01x04, J4 Conn_01x04, J5 Conn_01x04, J6 USB4105-GF-A-060, Q1 TPRT9013-33GB, SW2 SW_SPST, U1 BMP581, U2 MP9943GQ-Z, U3 USBLC6-2P6, U4 MP9943GQ-Z, Y2 X322525MOB4SI

Commit message: power planes
Connections:
- net +3.3v is gone; now on net +3.3V: IC3.8 (VCC), R16.1, R17.1
Changed lines of the file:
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@@
 			)
 		)
-		(property "Value" "+3.3v"
-			(at 36.83 238.76 0)
+		(property "Value" "+3.3V"
+			(at 39.37 242.5699 0)
 			(effects
 				(font
 					(size 1.27 1.27)
 				)
+				(justify left)
 			)
 		)

Commit message: power planes
Connections:
- net GNDREF is gone; now on net GND: C1.2, C10.2, C11.2, C13.2, C14.2, C15.2, C16.2, C19.2, C2.2, C20.2, C21.2, C22.2, C23.1, C24.1, C25.1, C26.1, C27.1, C28.1, C29.1, C3.2, C30.1, C31.1, C32.1, C35.1, C36.1, C4.2, C6.2, C7.2, C8.2, C9.2, D1.6 (GND), IC2.12 (VSSA), IC2.18 (VSS_1), IC2.31 (VSS_2), IC2.47 (VSS_3), IC2.63 (VSS_4), IC3.4 (GND), J1.3 (Pin_3), J2.7 (Pin_7), J3.1 (Pin_1), J4.1 (Pin_1), J5.1 (Pin_1), Q1.2 (GND), R11.1, R12.1, R13.1, R20.1, R22.1, R8.1, U1.3 (VSS_1), U1.5 (SDO), U1.6 (CSB), U1.8 (VSS_2), U1.9 (VSS_3), U2.5 (GND), U3.2 (GND), U4.5 (GND), Y2.3 (CRYSTAL__2), Y2.4 (GND_2)
- net +3.3V: no longer IC3.8 (VCC), R16.1, R17.1
- new net +3.3v: IC3.8 (VCC), R16.1, R17.1
Changed lines of the file:
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@@
 	(wire
 		(pts
+			(xy 15.24 33.02) (xy 17.78 33.02)
+		)
+		(stroke
+			(width 0)
+			(type default)
+		)
+	)
+	(wire
+		(pts
 			(xy 363.22 200.66) (xy 372.11 200.66)
 		)
@@
 	(wire
 		(pts
+			(xy 92.71 33.02) (xy 96.52 33.02)
+		)
+		(stroke
+			(width 0)
+			(type default)
+		)
+	)
+	(wire
+		(pts
 			(xy 353.06 109.22) (xy 382.27 109.22)
 		)
@@
 	(wire
 		(pts
-			(xy 96.52 30.48) (xy 96.52 44.45)
+			(xy 96.52 33.02) (xy 96.52 44.45)
 		)
 		(stroke
@@
 	(symbol
 		(lib_id "power:GNDREF")
+		(at 17.78 33.02 0)
+		(unit 1)
+		(exclude_from_sim no)
+		(in_bom yes)
+		(on_board yes)
+		(dnp no)
+		(property "Reference" "#PWR038"
+			(at 17.78 39.37 0)
+			(effects
+				(font
+					(size 1.27 1.27)
+				)
+				(hide yes)
+			)
+		)
+		(property "Value" "GNDREF"
+			(at 24.13 34.798 0)
+			(effects
+				(font
+					(size 1.27 1.27)
+				)
+			)
+		)
+		(property "Footprint" ""
+			(at 17.78 33.02 0)
+			(effects
+				(font
+					(size 1.27 1.27)
+				)
+				(hide yes)
+			)
+		)
+		(property "Datasheet" ""
+			(at 17.78 33.02 0)
+			(effects
+				(font
+					(size 1.27 1.27)
+				)
+				(hide yes)
+			)
+		)
+		(property "Description" "Power symbol creates a global label with name \"GNDREF\" , reference supply ground"
+			(at 17.78 33.02 0)
+			(effects
+				(font
+					(size 1.27 1.27)
+				)
+				(hide yes)
+			)
+		)
+		(pin "1"
+		)
+		(instances
+			(project ""
+				(path "/872311d7-35d2-44c4-a32c-18d15c37103e"
+					(reference "#PWR038")
+					(unit 1)
+				)
+			)
+		)
+	)
+	(symbol
+		(lib_id "power:GNDREF")
 		(at 278.13 58.42 0)
 		(unit 1)
@@
 			)
 		)
-		(property "Value" "+3.3V"
-			(at 39.37 242.5699 0)
+		(property "Value" "+3.3v"
+			(at 36.83 238.76 0)
 			(effects
 				(font
 					(size 1.27 1.27)
 				)
-				(justify left)
 			)
 		)
@@
 	)
 	(symbol
-		(lib_id "power:GND")
-		(at 15.24 33.02 180)
-		(unit 1)
-		(exclude_from_sim no)
-		(in_bom yes)
-		(on_board yes)
-		(dnp no)
-		(fields_autoplaced yes)
-		(property "Reference" "#PWR038"
-			(at 15.24 26.67 0)
-			(effects
-				(font
-					(size 1.27 1.27)
-				)
-				(hide yes)
-			)
-		)
-		(property "Value" "GND"
-			(at 15.24 27.94 0)
-			(effects
-				(font
-					(size 1.27 1.27)
-				)
-			)
-		)
-		(property "Footprint" ""
-			(at 15.24 33.02 0)
-			(effects
-				(font
-					(size 1.27 1.27)
-				)
-				(hide yes)
-			)
-		)
-		(property "Datasheet" ""
-			(at 15.24 33.02 0)
-			(effects
-				(font
-					(size 1.27 1.27)
-				)
-				(hide yes)
-			)
-		)
-		(property "Description" "Power symbol creates a global label with name \"GND\" , ground"
-			(at 15.24 33.02 0)
-			(effects
-				(font
-					(size 1.27 1.27)
-				)
-				(hide yes)
-			)
-		)
-		(pin "1"
-		)
-		(instances
-			(project "flight_controller"
-				(path "/872311d7-35d2-44c4-a32c-18d15c37103e"
-					(reference "#PWR038")
-					(unit 1)
-				)
-			)
-		)
-	)
-	(symbol
 		(lib_id "Device:C")
 		(at 100.33 120.65 0)
@@
 	)
 	(symbol
-		(lib_id "power:GND")
-		(at 96.52 30.48 180)
-		(unit 1)
-		(exclude_from_sim no)
-		(in_bom yes)
-		(on_board yes)
-		(dnp no)
-		(property "Reference" "#PWR058"
-			(at 96.52 24.13 0)
-			(effects
-				(font
-					(size 1.27 1.27)
-				)
-				(hide yes)
-			)
-		)
-		(property "Value" "GND"
-			(at 95.25 26.416 0)
-			(effects
-				(font
-					(size 1.27 1.27)
-				)
-			)
-		)
-		(property "Footprint" ""
-			(at 96.52 30.48 0)
-			(effects
-				(font
-					(size 1.27 1.27)
-				)
-				(hide yes)
-			)
-		)
-		(property "Datasheet" ""
-			(at 96.52 30.48 0)
-			(effects
-				(font
-					(size 1.27 1.27)
-				)
-				(hide yes)
-			)
-		)
-		(property "Description" "Power symbol creates a global label with name \"GND\" , ground"
-			(at 96.52 30.48 0)
-			(effects
-				(font
-					(size 1.27 1.27)
-				)
-				(hide yes)
-			)
-		)
-		(pin "1"
-		)
-		(instances
-			(project "flight_controller"
-				(path "/872311d7-35d2-44c4-a32c-18d15c37103e"
-					(reference "#PWR058")
-					(unit 1)
-				)
-			)
-		)
-	)
-	(symbol
 		(lib_id "power:VCC")
 		(at 60.96 160.02 0)
@@
 					(unit 1)
 				)
+			)
+		)
+	)
+	(symbol
+		(lib_id "power:GNDREF")
+		(at 92.71 33.02 0)
+		(unit 1)
+		(exclude_from_sim no)
+		(in_bom yes)
+		(on_board yes)
+		(dnp no)
+		(property "Reference" "#PWR055"
+			(at 92.71 39.37 0)
+			(effects
+				(font
+					(size 1.27 1.27)
+				)
+				(hide yes)
+			)
+		)
+		(property "Value" "GNDREF"
+			(at 86.36 34.29 0)
+			(effects
+				(font
+					(size 1.27 1.27)
+				)
+			)
+		)
+		(property "Footprint" ""
+			(at 92.71 33.02 0)
+			(effects
+				(font
+					(size 1.27 1.27)
+				)
+				(hide yes)
+			)
+		)
+		(property "Datasheet" ""
+			(at 92.71 33.02 0)
+			(effects
+				(font
+					(size 1.27 1.27)
+				)
+				(hide yes)
+			)
+		)
+		(property "Description" "Power symbol creates a global label with name \"GNDREF\" , reference supply ground"
+			(at 92.71 33.02 0)
+			(effects
+				(font
+					(size 1.27 1.27)
+				)
+				(hide yes)
+			)
+		)
+		(pin "1"
+		)
+		(instances
+			(project "flight_controller"
+				(path "/872311d7-35d2-44c4-a32c-18d15c37103e"
+					(reference "#PWR055")
+					(unit 1)
+				)

Commit message: stackup
Connections:
- net +3.3v is gone; now on net +3.3V: IC3.8 (VCC), R16.1, R17.1
Changed lines of the file:
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@@
 			)
 		)
-		(property "Value" "+3.3v"
-			(at 36.83 238.76 0)
+		(property "Value" "+3.3V"
+			(at 39.37 242.5699 0)
 			(effects
 				(font
 					(size 1.27 1.27)
 				)
+				(justify left)
 			)
 		)

Commit message: fix errors
Connections:
- net USB_DN: no longer IC2.44 (PA11), R9.2
- net USB_DP: no longer IC2.45 (PA12), R10.2
- new net USB_D_DN: IC2.44 (PA11), R9.2
- new net USB_D_DP: IC2.45 (PA12), R10.2
Changed lines of the file:
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@@
 		)
 	)
-	(label "USB_DN"
+	(label "USB_D_DN"
 		(at 339.09 99.06 180)
 		(effects
@@
 		)
 	)
-	(label "USB_DP"
+	(label "USB_D_DP"
 		(at 339.09 96.52 180)
 		(effects
@@
 		)
 	)
-	(label "USB_DP"
+	(label "USB_D_DP"
 		(at 299.72 36.83 0)
 		(effects
@@
 		)
 	)
-	(label "USB_DN"
+	(label "USB_D_DN"
 		(at 299.72 34.29 0)
 		(effects

Commit message: fix errors
Parts:
- D3, D4, D5: footprint Diode_SMD:D_SOD-523 -> LED_SMD:LED_0603_1608Metric
Changed lines of the file:
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@@
 			)
 		)
-		(property "Footprint" "Diode_SMD:D_SOD-523"
+		(property "Footprint" "LED_SMD:LED_0603_1608Metric"
 			(at 315.595 233.68 0)
 			(effects
@@
 			)
 		)
-		(property "Footprint" "Diode_SMD:D_SOD-523"
+		(property "Footprint" "LED_SMD:LED_0603_1608Metric"
 			(at 297.815 233.68 0)
 			(effects
@@
 			)
 		)
-		(property "Footprint" "Diode_SMD:D_SOD-523"
+		(property "Footprint" "LED_SMD:LED_0603_1608Metric"
 			(at 280.035 234.95 0)
 			(effects

Commit message: fix errors
Parts:
- D3: value 1N4148WT -> YLED0603YG
- D4: value 1N4148WT -> YLED0603R
- D5: value 1N4148WT -> YLED0603G
- R13: value 470Ω -> 33Ω
Changed lines of the file:
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@@
 			)
 		)
-		(property "Value" "470Ω"
+		(property "Value" "33Ω"
 			(at 316.23 242.316 0)
 			(effects
@@
 			)
 		)
-		(property "Value" "1N4148WT"
+		(property "Value" "YLED0603G"
 			(at 313.69 234.9499 90)
 			(effects
@@
 			)
 		)
-		(property "Value" "1N4148WT"
+		(property "Value" "YLED0603R"
 			(at 295.91 234.9499 90)
 			(effects
@@
 			)
 		)
-		(property "Value" "1N4148WT"
+		(property "Value" "YLED0603YG"
 			(at 278.13 236.2199 90)
 			(effects

Commit message: fix errors
Parts:
- R14: value R2 5.1KΩ -> 5.1KΩ
- R15: value R1 5.1KΩ -> 5.1KΩ
Changed lines of the file:
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@@
 			)
 		)
-		(property "Value" "R2 5.1KΩ"
+		(property "Value" "5.1KΩ"
 			(at 20.32 42.164 90)
 			(effects
@@
 			)
 		)
-		(property "Value" "R1 5.1KΩ"
+		(property "Value" "5.1KΩ"
 			(at 91.186 42.164 90)
 			(effects

Commit message: fix errors
Parts:
- J3, J4, J5: now left out of the parts list
Changed lines of the file:
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@@
 		(unit 1)
 		(exclude_from_sim no)
-		(in_bom yes)
+		(in_bom no)
 		(on_board yes)
 		(dnp no)
@@
 		(unit 1)
 		(exclude_from_sim no)
-		(in_bom yes)
+		(in_bom no)
 		(on_board yes)
 		(dnp no)
@@
 		(unit 1)
 		(exclude_from_sim no)
-		(in_bom yes)
+		(in_bom no)
 		(on_board yes)
 		(dnp no)
