File: hardware/flight_controller.kicad_pcb (KiCad board)
At the start: 6 copper layers, 50 x 50 mm, 81 parts, among them IC2 STM32F722RET6, IC3 W25Q128JVSIQ, J1 Conn_01x03, J2 Conn_01x08, J3 Conn_01x04, J4 Conn_01x04, J5 Conn_01x04, J6 USB4105-GF-A-060, Q1 TPRT9013-33GB, SW2 SW_SPST, U1 BMP581, U2 MP9943GQ-Z, U3 USBLC6-2P6, U4 MP9943GQ-Z, Y2 X322525MOB4SI

Commit message: fix errors
Routing:
- net +5V: track 7.90 -> 9.10 mm, vias 4 -> 5
- net +3.3V: track 51.8 -> 52.6 mm
- net GNDREF: track 3.18 -> 3.81 mm
Changed lines of the file:
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@@
 		(sheetname "/")
 		(sheetfile "flight_controller.kicad_sch")
-		(solder_mask_margin -0.02)
-		(attr smd allow_soldermask_bridges)
+		(solder_mask_margin -0.05)
+		(clearance 0)
+		(attr smd)
 		(fp_line
 			(start 4.47 -2.65)
@@
 			(pinfunction "GND")
 			(pintype "power_in")
-			(solder_mask_margin 0.102)
+			(solder_mask_margin 0.001)
 		)
 		(pad "A4_B9" smd rect
@@
 			(pinfunction "VBUS")
 			(pintype "power_in")
-			(solder_mask_margin 0.102)
+			(solder_mask_margin 0.001)
 		)
 		(pad "A5" smd rect
@@
 			(pinfunction "CC1")
 			(pintype "bidirectional")
-			(solder_mask_margin 0.102)
+			(solder_mask_margin 0.001)
 		)
 		(pad "A6" smd rect
@@
 			(pinfunction "DP1")
 			(pintype "bidirectional")
-			(solder_mask_margin 0.102)
+			(solder_mask_margin 0.001)
 		)
 		(pad "A7" smd rect
@@
 			(pinfunction "DN1")
 			(pintype "bidirectional")
-			(solder_mask_margin 0.102)
+			(solder_mask_margin 0.001)
 		)
 		(pad "A8" smd rect
@@
 			(pinfunction "SBU1")
 			(pintype "bidirectional+no_connect")
-			(solder_mask_margin 0.102)
+			(solder_mask_margin 0.01)
 		)
 		(pad "B1_A12" smd rect
@@
 			(pinfunction "GND")
 			(pintype "power_in")
-			(solder_mask_margin 0.102)
+			(solder_mask_margin 0.01)
 		)
 		(pad "B4_A9" smd rect
@@
 			(pinfunction "VBUS")
 			(pintype "power_in")
-			(solder_mask_margin 0.102)
+			(solder_mask_margin 0.01)
 		)
 		(pad "B5" smd rect
@@
 			(pinfunction "CC2")
 			(pintype "bidirectional")
-			(solder_mask_margin 0.102)
+			(solder_mask_margin 0.001)
 		)
 		(pad "B6" smd rect
@@
 			(pinfunction "DP2")
 			(pintype "bidirectional")
-			(solder_mask_margin 0.102)
+			(solder_mask_margin 0.001)
 		)
 		(pad "B7" smd rect
@@
 			(pinfunction "DN2")
 			(pintype "bidirectional")
-			(solder_mask_margin 0.102)
+			(solder_mask_margin 0.001)
 		)
 		(pad "B8" smd rect
@@
 			(pinfunction "SBU2")
 			(pintype "bidirectional+no_connect")
-			(solder_mask_margin 0.102)
+			(solder_mask_margin 0.001)
 		)
 		(pad "SH1" thru_hole oval
@@
 	)
 	(segment
+		(start 173.322404 121.272404)
+		(end 172.67497 121.272404)
+		(width 0.2)
+		(layer "F.Cu")
+		(net 5)
+	)
+	(segment
 		(start 180.88894 95.269912)
 		(end 179.941109 96.217743)
@@
 	)
 	(segment
+		(start 173.028891 114.75543)
+		(end 173.278891 115.00543)
+		(width 0.2)
+		(layer "F.Cu")
+		(net 5)
+	)
+	(segment
 		(start 171.138624 105.911376)
 		(end 170.85 106.2)
@@
 	)
 	(segment
-		(start 173.322404 121.272404)
-		(end 173.55 121.5)
-		(width 0.2)
-		(layer "F.Cu")
-		(net 5)
-	)
-	(segment
 		(start 169.5 120.75)
 		(end 169.5 119.774013)
@@
 	)
 	(segment
+		(start 173.394808 121.2)
+		(end 173.322404 121.272404)
+		(width 0.2)
+		(layer "F.Cu")
+		(net 5)
+	)
+	(segment
+		(start 173.75 121.2)
+		(end 173.394808 121.2)
+		(width 0.2)
+		(layer "F.Cu")
+		(net 5)
+	)
+	(segment
 		(start 198.25 94)
 		(end 196.95 95.3)
@@
 	)
 	(segment
-		(start 172.67497 121.272404)
-		(end 173.322404 121.272404)
-		(width 0.2)
-		(layer "F.Cu")
-		(net 5)
-	)
-	(segment
 		(start 164.85 87.4)
 		(end 164.85 87.025972)
@@
 		(net 5)
 	)
+	(segment
+		(start 173.278891 115.00543)
+		(end 173.553891 115.00543)
+		(width 0.2)
+		(layer "F.Cu")
+		(net 5)
+	)
 	(via
 		(at 170.85 106.2)
@@
 	)
 	(via
-		(at 173.55 121.5)
+		(at 173.75 121.2)
 		(size 0.5)
 		(drill 0.3)
@@
 	)
 	(segment
-		(start 191.9075 113.9)
-		(end 192.516492 113.9)
+		(start 193.25 113.166492)
+		(end 193.25 109.8655)
 		(width 0.2)
 		(layer "F.Cu")
@@
 	)
 	(segment
-		(start 193.75 112.666492)
-		(end 193.75 110.3655)
+		(start 193.25 109.8655)
+		(end 192.4845 109.1)
 		(width 0.2)
 		(layer "F.Cu")
@@
 	)
 	(segment
-		(start 193.75 110.3655)
-		(end 192.4845 109.1)
-		(width 0.2)
+		(start 189.487512 109.1)
+		(end 191.9075 109.1)
+		(width 0.5)
 		(layer "F.Cu")
 		(net 11)
 	)
 	(segment
-		(start 189.487512 109.1)
-		(end 191.9075 109.1)
-		(width 0.5)
+		(start 191.9075 113.9)
+		(end 192.516492 113.9)
+		(width 0.2)
 		(layer "F.Cu")
 		(net 11)
@@
 	(segment
 		(start 192.516492 113.9)
-		(end 193.75 112.666492)
+		(end 193.25 113.166492)
 		(width 0.2)
 		(layer "F.Cu")
@@
 	)
 	(segment
+		(start 174.578891 113.75543)
+		(end 174.303891 113.75543)
+		(width 0.1)
+		(layer "F.Cu")
+		(net 12)
+	)
+	(segment
 		(start 191.9075 115.245)
 		(end 192.4825 115.82)
@@
 		(net 12)
 	)
+	(segment
+		(start 174.303891 113.75543)
+		(end 174.053891 113.50543)
+		(width 0.1)
+		(layer "F.Cu")
+		(net 12)
+	)
 	(via
 		(at 172.093722 111.61861)
@@
 	)
 	(via
-		(at 184.300212 114.587619)
+		(at 173.914779 102.286424)
 		(size 0.4)
 		(drill 0.2)
@@
 	)
 	(via
-		(at 173.914779 102.286424)
+		(at 198.113794 127.590761)
 		(size 0.4)
 		(drill 0.2)
@@
 	)
 	(via
-		(at 198.113794 127.590761)
+		(at 174.287852 96.860528)
 		(size 0.4)
 		(drill 0.2)
@@
 	)
 	(via
-		(at 174.287852 96.860528)
+		(at 166.65 115.1)
 		(size 0.4)
 		(drill 0.2)
@@
 	)
 	(via
-		(at 166.65 115.1)
+		(at 174.441162 112.51247)
 		(size 0.4)
 		(drill 0.2)
@@
 	)
 	(via
-		(at 175.104045 123.054045)
+		(at 175.028393 123.003314)
 		(size 0.4)
 		(drill 0.2)
@@
 	)
 	(via
-		(at 174.08252 113.983146)
+		(at 174.118961 115.605162)
 		(size 0.4)
 		(drill 0.2)
@@
 	)
 	(via
-		(at 181.206469 115.037922)
+		(at 181.547594 115.204811)
 		(size 0.4)
 		(drill 0.2)
@@
 	)
 	(segment
-		(start 174.578891 114.25543)
-		(end 174.993391 114.25543)
+		(start 174.25 111.25)
+		(end 174.25 110.394134)
 		(width 0.2)
 		(layer "F.Cu")
@@
 	)
 	(segment
-		(start 175.25 112.25)
-		(end 174.25 111.25)
+		(start 174.578891 114.25543)
+		(end 174.993391 114.25543)
 		(width 0.2)
 		(layer "F.Cu")
@@
 	)
 	(segment
-		(start 174.25 110.394134)
-		(end 176.068993 108.575141)
+		(start 175.25 113.998821)
+		(end 175.25 112.25)
 		(width 0.2)
 		(layer "F.Cu")
@@
 	)
 	(segment
-		(start 174.25 111.25)
-		(end 174.25 110.394134)
+		(start 174.993391 114.25543)
+		(end 175.25 113.998821)
 		(width 0.2)
 		(layer "F.Cu")
@@
 	)
 	(segment
-		(start 175.25 113.998821)
-		(end 175.25 112.25)
+		(start 175.25 112.25)
+		(end 174.25 111.25)
 		(width 0.2)
 		(layer "F.Cu")
@@
 	)
 	(segment
-		(start 174.993391 114.25543)
-		(end 175.25 113.998821)
+		(start 174.25 110.394134)
+		(end 176.068993 108.575141)
 		(width 0.2)
 		(layer "F.Cu")
@@
 	)
 	(segment
+		(start 171.95 123.3)
+		(end 172 123.35)
+		(width 0.1)
+		(layer "F.Cu")
+		(net 51)
+	)
+	(segment
+		(start 171.4 123.25)
+		(end 171.9 123.25)
+		(width 0.5)
+		(layer "F.Cu")
+		(net 51)
+	)
+	(segment
 		(start 187.663236 113.413236)
 		(end 188.05 113.8)
@@
 	)
 	(segment
+		(start 171.9 123.25)
+		(end 171.95 123.3)
+		(width 0.1)
+		(layer "F.Cu")
+		(net 51)
+	)
+	(segment
 		(start 167.248971 123.393211)
 		(end 168.176091 123.393211)
@@
 		(net 51)
 	)
+	(segment
+		(start 171.95 123.3)
+		(end 172.35 123.7)
+		(width 0.5)
+		(layer "F.Cu")
+		(net 51)
+	)
 	(via
 		(at 188.05 115.1)
@@
 		(layers "F.Cu" "B.Cu")
 		(net 51)
+	)
+	(via
+		(at 172.35 123.7)
+		(size 0.4)
+		(drill 0.2)
+		(layers "F.Cu" "B.Cu")
+		(net 51)

Commit message: fix errors
Parts:
- D3, D4, D5: footprint Diode_SMD:D_SOD-523 -> LED_SMD:LED_0603_1608Metric
