File: hardware/flight_controller.kicad_pcb (KiCad board)
At the start: 6 copper layers, 50 x 50 mm, 81 parts, among them IC2 STM32F722RET6, IC3 W25Q128JVSIQ, J1 Conn_01x03, J2 Conn_01x08, J3 Conn_01x04, J4 Conn_01x04, J5 Conn_01x04, J6 USB4105-GF-A-060, Q1 TPRT9013-33GB, SW2 SW_SPST, U1 BMP581, U2 MP9943GQ-Z, U3 USBLC6-2P6, U4 MP9943GQ-Z, Y2 X322525MOB4SI

Commit message: fix errors
Parts:
- D3: value 1N4148WT -> YLED0603YG
- D4: value 1N4148WT -> YLED0603R
- D5: value 1N4148WT -> YLED0603G
- R13: value 470Ω -> 33Ω
Changed lines of the file:
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@@
 			)
 		)
-		(property "Value" "1N4148WT"
+		(property "Value" "YLED0603YG"
 			(at 0 1.43 0)
 			(layer "F.Fab")
@@
 			)
 		)
-		(property "Value" "1N4148WT"
+		(property "Value" "YLED0603R"
 			(at 0 1.43 0)
 			(layer "F.Fab")
@@
 			)
 		)
-		(property "Value" "470Ω"
+		(property "Value" "33Ω"
 			(at 0 1 0)
 			(layer "F.Fab")
@@
 			)
 		)
-		(property "Value" "1N4148WT"
+		(property "Value" "YLED0603G"
 			(at 0 1.43 0)
 			(layer "F.Fab")

Commit message: fix errors
Parts:
- FB1: value FerriteBead -> C141723
Changed lines of the file:
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@@
 		(sheetname "/")
 		(sheetfile "flight_controller.kicad_sch")
-		(attr through_hole exclude_from_pos_files)
+		(attr through_hole exclude_from_pos_files exclude_from_bom)
 		(fp_line
 			(start -1.38 -1.38)
@@
 		(sheetname "/")
 		(sheetfile "flight_controller.kicad_sch")
-		(attr through_hole exclude_from_pos_files)
+		(attr through_hole exclude_from_pos_files exclude_from_bom)
 		(fp_line
 			(start -1.38 -1.38)
@@
 		(sheetname "/")
 		(sheetfile "flight_controller.kicad_sch")
-		(attr through_hole exclude_from_pos_files)
+		(attr through_hole exclude_from_pos_files exclude_from_bom)
 		(fp_line
 			(start -1.38 -1.38)
@@
 				(font
 					(size 0.5 0.5)
-					(thickness 0.15)
+					(thickness 0.125)
 				)
 			)
 		)
-		(property "Value" "FerriteBead"
+		(property "Value" "C141723"
 			(at 0 1.43 45)
 			(layer "F.Fab")
@@
 		(sheetname "/")
 		(sheetfile "flight_controller.kicad_sch")
-		(attr through_hole exclude_from_pos_files)
+		(attr through_hole exclude_from_pos_files exclude_from_bom)
 		(fp_line
 			(start -0.745 -0.735)

Commit message: fix errors
Parts:
- FB1: value C141723 -> FCM1608KF-601T03
- J2: value Conn_01x08 -> JST SM08B-SRSS-TB(LF)(SN)
- R14: value R2 5.1KΩ -> 5.1KΩ
- R15: value R1 5.1KΩ -> 5.1KΩ
- R16, R17: value 10k -> 10KΩ
- SW2: value SW_SPST -> KMR221GLFS
Changed lines of the file:
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@@
 			)
 		)
-		(property "Value" "R1 5.1KΩ"
+		(property "Value" "5.1KΩ"
 			(at 0 1 90)
 			(layer "F.Fab")
@@
 			)
 		)
-		(property "Value" "C141723"
+		(property "Value" "FCM1608KF-601T03"
 			(at 0 1.43 45)
 			(layer "F.Fab")
@@
 			)
 		)
-		(property "Value" "10k"
+		(property "Value" "10KΩ"
 			(at 0 1 90)
 			(layer "F.Fab")
@@
 		(tags "Undefined or Miscellaneous")
 		(property "Reference" "U1"
-			(at 0 0 90)
+			(at 0.014621 2.018483 90)
 			(layer "F.SilkS")
 			(effects
@@
 			)
 		)
-		(property "Value" "10k"
+		(property "Value" "10KΩ"
 			(at 0 1 90)
 			(layer "F.Fab")
@@
 			)
 		)
-		(property "Value" "SW_SPST"
+		(property "Value" "KMR221GLFS"
 			(at 0 2.55 90)
 			(layer "F.Fab")
@@
 			)
 		)
-		(property "Value" "Conn_01x08"
+		(property "Value" "JST SM08B-SRSS-TB(LF)(SN)"
 			(at 0 3.98 0)
 			(layer "F.Fab")
@@
 			)
 		)
-		(property "Value" "R2 5.1KΩ"
+		(property "Value" "5.1KΩ"
 			(at 0 1 90)
 			(layer "F.Fab")

Commit message: fix errors
Parts:
- C30: footprint Capacitor_SMD:C_0201_0603Metric -> Capacitor_SMD:C_0402_1005Metric
Changed lines of the file:
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@@
 		)
 	)
-	(footprint "Capacitor_SMD:C_0201_0603Metric"
+	(footprint "Capacitor_SMD:C_0402_1005Metric"
 		(layer "F.Cu")
 		(at 168.836889 119.430902)
-		(descr "Capacitor SMD 0201 (0603 Metric), square (rectangular) end terminal, IPC-7351 nominal, (Body size source: https://www.vishay.com/docs/20052/crcw0201e3.pdf), generated with kicad-footprint-generator")
+		(descr "Capacitor SMD 0402 (1005 Metric), square (rectangular) end terminal, IPC-7351 nominal, (Body size source: IPC-SM-782 page 76, https://www.pcb-3d.com/wordpress/wp-content/uploads/ipc-sm-782a_amendment_1_and_2.pdf), generated with kicad-footprint-generator")
 		(tags "capacitor")
 		(property "Reference" "C30"
-			(at 0 -0.730902 0)
+			(at 0 -1.16 0)
 			(layer "F.SilkS")
 			(effects
@@
 		)
 		(property "Value" "10μF"
-			(at 0 1.05 0)
+			(at 0 1.16 0)
 			(layer "F.Fab")
 			(hide yes)
@@
 		(sheetfile "flight_controller.kicad_sch")
 		(attr smd)
+		(fp_line
+			(start -0.107836 -0.36)
+			(end 0.107836 -0.36)
+			(stroke
+				(width 0.12)
+				(type solid)
+			)
+			(layer "F.SilkS")
+		)
+		(fp_line
+			(start -0.107836 0.36)
+			(end 0.107836 0.36)
+			(stroke
+				(width 0.12)
+				(type solid)
+			)
+			(layer "F.SilkS")
+		)
 		(fp_rect
-			(start -0.7 -0.35)
-			(end 0.7 0.35)
+			(start -0.91 -0.46)
+			(end 0.91 0.46)
 			(stroke
 				(width 0.05)
@@
 		)
 		(fp_rect
-			(start -0.3 -0.15)
-			(end 0.3 0.15)
+			(start -0.5 -0.25)
+			(end 0.5 0.25)
 			(stroke
 				(width 0.1)
@@
 			(layer "F.Fab")
 		)
-		(pad "" smd roundrect
-			(at -0.345 0)
-			(size 0.318 0.36)
-			(layers "F.Paste")
-			(roundrect_rratio 0.25)
-		)
-		(pad "" smd roundrect
-			(at 0.345 0)
-			(size 0.318 0.36)
-			(layers "F.Paste")
-			(roundrect_rratio 0.25)
+		(fp_text user "${REFERENCE}"
+			(at 0 0 0)
+			(layer "F.Fab")
+			(effects
+				(font
+					(size 0.25 0.25)
+					(thickness 0.04)
+				)
+			)
 		)
 		(pad "1" smd roundrect
-			(at -0.32 0)
-			(size 0.46 0.4)
-			(layers "F.Cu" "F.Mask")
+			(at -0.48 0)
+			(size 0.56 0.62)
+			(layers "F.Cu" "F.Mask" "F.Paste")
 			(roundrect_rratio 0.25)
 			(net 12 "GNDREF")
@@
 		)
 		(pad "2" smd roundrect
-			(at 0.32 0)
-			(size 0.46 0.4)
-			(layers "F.Cu" "F.Mask")
+			(at 0.48 0)
+			(size 0.56 0.62)
+			(layers "F.Cu" "F.Mask" "F.Paste")
 			(roundrect_rratio 0.25)
 			(net 5 "+3.3V")
@@
 		)
 		(embedded_fonts no)
-		(model "${KICAD9_3DMODEL_DIR}/Capacitor_SMD.3dshapes/C_0201_0603Metric.step"
+		(model "${KICAD9_3DMODEL_DIR}/Capacitor_SMD.3dshapes/C_0402_1005Metric.step"
 			(offset
 				(xyz 0 0 0)
@@
 	)
 	(segment
-		(start 169.5 119.774013)
-		(end 169.156889 119.430902)
+		(start 170.108713 111.958713)
+		(end 170.05 111.9)
+		(width 0.2)
+		(layer "F.Cu")
+		(net 5)
+	)
+	(segment
+		(start 169.919098 119.430902)
+		(end 170.25 119.1)
 		(width 0.3)
 		(layer "F.Cu")
@@
 	)
 	(segment
-		(start 170.108713 111.958713)
-		(end 170.05 111.9)
-		(width 0.2)
+		(start 169.316889 119.430902)
+		(end 169.919098 119.430902)
+		(width 0.3)
 		(layer "F.Cu")
 		(net 5)
@@
 	)
 	(segment
-		(start 168.3 120.75)
-		(end 168.15 120.9)
+		(start 169.5 120.75)
+		(end 169.5 119.774013)
 		(width 0.3)
 		(layer "F.Cu")
@@
 	)
 	(segment
-		(start 169.5 120.75)
-		(end 169.5 119.774013)
+		(start 169.5 119.774013)
+		(end 169.316889 119.590902)
 		(width 0.3)
 		(layer "F.Cu")
@@
 	)
 	(segment
+		(start 169.316889 119.590902)
+		(end 169.316889 119.430902)
+		(width 0.3)
+		(layer "F.Cu")
+		(net 5)
+	)
+	(segment
 		(start 173.75 121.2)
 		(end 173.394808 121.2)
@@
 	)
 	(segment
-		(start 169.5 120.75)
-		(end 168.3 120.75)
-		(width 0.3)
-		(layer "F.Cu")
-		(net 5)
-	)
-	(segment
 		(start 186.550325 103.6912)
 		(end 186.550325 103.600325)
@@
 	)
 	(via
-		(at 168.15 120.9)
+		(at 174.513909 118.263909)
 		(size 0.5)
 		(drill 0.3)
@@
 	)
 	(via
-		(at 174.513909 118.263909)
-		(size 0.5)
-		(drill 0.3)
+		(at 170.25 119.1)
+		(size 0.4)
+		(drill 0.2)
 		(layers "F.Cu" "B.Cu")
 		(net 5)

Commit message: resizing
Parts:
- C27, C28, C29, C32, C8, C9: footprint Capacitor_SMD:C_0201_0603Metric -> Capacitor_SMD:C_0603_1608Metric
- C30: footprint Capacitor_SMD:C_0402_1005Metric -> Capacitor_SMD:C_0805_2012Metric
- R1, R10, R11, R12, R13, R14, R15, R16, R17, R18, R19, R2, R20, R21, R22, R3, R4, R5, R6, R7, R8, R9: footprint Resistor_SMD:R_01005_0402Metric -> Resistor_SMD:R_0402_1005Metric
- moved C8 5.16 mm to (167.8, 119.4)
- moved C30 1.73 mm to (170.4, 118.7), turned to 180 degrees
- moved C29 1.61 mm to (188.4, 104.0), turned to 90 degrees
- moved C25 1.33 mm to (177.4, 112.7), turned to 90 degrees
- moved R3 1.31 mm to (155.8, 98.2), turned to 180 degrees
- moved C4 0.89 mm to (155.9, 99.4)
- moved R4 0.83 mm to (155.8, 100.6)
- moved C27 0.78 mm to (175.8, 93.3)
- moved R19 0.72 mm to (175.0, 123.2), turned to 0 degrees
- moved C28 0.72 mm to (169.0, 99.3)
- moved C9 0.62 mm to (167.8, 122.6)
- moved R6 0.60 mm to (158.9, 108.2)
- moved R5 0.58 mm to (155.9, 101.8)
- moved C32 0.52 mm to (175.8, 110.8)
- moved R12 0.45 mm to (194.9, 96.5)
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Routing:
- net +3.3V: track 52.2 -> 60.7 mm, vias 15 -> 14
- net /BMP_SDI: track 7.37 -> 9.59 mm, vias 0 -> 2
- net Net-(U2-VCC): track 3.14 -> 4.81 mm
- net GNDREF: track 3.81 -> 5.33 mm, vias 34 -> 35
- net +5VBAT: track 10.3 -> 8.88 mm
- net /BOOT: track 21.4 -> 22.5 mm
- net Net-(U4-FB): track 9.20 -> 10.3 mm
- net Net-(U2-EN/SYNC): track 1.79 -> 2.64 mm
- net Net-(R19-Pad2): track 1.47 -> 2.20 mm
- net Net-(R6-Pad2): track 1.62 -> 2.23 mm
- net +5V: track 9.10 -> 9.64 mm
- net Net-(C5-Pad2): track 1.13 -> 1.64 mm

Commit message: resizing
Parts:
- moved R1 0.82 mm to (184.4, 120.5)
- moved R2 0.59 mm to (182.2, 120.5)
- moved C10 0.58 mm to (183.3, 120.5)
- moved R18 0.40 mm to (181.2, 120.5)
Routing:
- net Net-(U4-VCC): track 2.91 -> 3.81 mm
Changed lines of the file:
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@@
 	(footprint "Capacitor_SMD:C_0402_1005Metric"
 		(layer "F.Cu")
-		(at 180.038651 120.546412 90)
+		(at 180.038651 120.52 90)
 		(descr "Capacitor SMD 0402 (1005 Metric), square (rectangular) end terminal, IPC-7351 nominal, (Body size source: IPC-SM-782 page 76, https://www.pcb-3d.com/wordpress/wp-content/uploads/ipc-sm-782a_amendment_1_and_2.pdf), generated with kicad-footprint-generator")
 		(tags "capacitor")
 		(property "Reference" "C12"
-			(at 1.446412 0.011349 270)
+			(at 1.746412 0.011349 270)
 			(layer "F.SilkS")
 			(effects
@@
 	(footprint "Resistor_SMD:R_0402_1005Metric"
 		(layer "F.Cu")
-		(at 180.990411 120.878632 90)
+		(at 181.15 120.51 90)
 		(descr "Resistor SMD 0402 (1005 Metric), square (rectangular) end terminal, IPC-7351 nominal, (Body size source: IPC-SM-782 page 72, https://www.pcb-3d.com/wordpress/wp-content/uploads/ipc-sm-782a_amendment_1_and_2.pdf), generated with kicad-footprint-generator")
 		(tags "resistor")
 		(property "Reference" "R18"
-			(at 0 -1.17 90)
+			(at 1.71 0.059589 90)
 			(layer "F.SilkS")
 			(effects
 				(font
-					(size 1 1)
-					(thickness 0.15)
+					(size 0.5 0.5)
+					(thickness 0.125)
 				)
 			)
@@
 			(at 0 1.17 90)
 			(layer "F.Fab")
+			(hide yes)
 			(effects
 				(font
@@
 	(footprint "Resistor_SMD:R_0402_1005Metric"
 		(layer "F.Cu")
-		(at 183.673554 120.861627 90)
+		(at 184.409589 120.49 90)
 		(descr "Resistor SMD 0402 (1005 Metric), square (rectangular) end terminal, IPC-7351 nominal, (Body size source: IPC-SM-782 page 72, https://www.pcb-3d.com/wordpress/wp-content/uploads/ipc-sm-782a_amendment_1_and_2.pdf), generated with kicad-footprint-generator")
 		(tags "resistor")
 		(property "Reference" "R1"
-			(at 0 -1.17 90)
+			(at 1.51 0 90)
 			(layer "F.SilkS")
 			(effects
 				(font
-					(size 1 1)
-					(thickness 0.15)
+					(size 0.5 0.5)
+					(thickness 0.125)
 				)
 			)
@@
 			(at 0 1.17 90)
 			(layer "F.Fab")
+			(hide yes)
 			(effects
 				(font
@@
 	(footprint "Resistor_SMD:R_0402_1005Metric"
 		(layer "F.Cu")
-		(at 181.777447 120.876077 -90)
+		(at 182.237036 120.51 -90)
 		(descr "Resistor SMD 0402 (1005 Metric), square (rectangular) end terminal, IPC-7351 nominal, (Body size source: IPC-SM-782 page 72, https://www.pcb-3d.com/wordpress/wp-content/uploads/ipc-sm-782a_amendment_1_and_2.pdf), generated with kicad-footprint-generator")
 		(tags "resistor")
 		(property "Reference" "R2"
-			(at 0 -1.17 270)
+			(at -1.51 -0.072553 90)
 			(layer "F.SilkS")
 			(effects
 				(font
-					(size 1 1)
-					(thickness 0.15)
+					(size 0.5 0.5)
+					(thickness 0.125)
 				)
 			)
 		)
 		(property "Value" "100KΩ"
-			(at 0 1.17 270)
+			(at 0 1.17 90)
 			(layer "F.Fab")
+			(hide yes)
 			(effects
 				(font
@@
 		)
 		(property "Datasheet" "~"
-			(at 0 0 270)
+			(at 0 0 90)
 			(layer "F.Fab")
 			(hide yes)
@@
 		)
 		(property "Description" "Resistor"
-			(at 0 0 270)
+			(at 0 0 90)
 			(layer "F.Fab")
 			(hide yes)
@@
 		)
 		(fp_text user "${REFERENCE}"
-			(at 0 0 270)
+			(at 0 0 90)
 			(layer "F.Fab")
 			(effects
@@
 	(footprint "Capacitor_SMD:C_0402_1005Metric"
 		(layer "F.Cu")
-		(at 182.734346 120.547011 90)
+		(at 183.309589 120.52 90)
 		(descr "Capacitor SMD 0402 (1005 Metric), square (rectangular) end terminal, IPC-7351 nominal, (Body size source: IPC-SM-782 page 76, https://www.pcb-3d.com/wordpress/wp-content/uploads/ipc-sm-782a_amendment_1_and_2.pdf), generated with kicad-footprint-generator")
 		(tags "capacitor")
 		(property "Reference" "C10"
-			(at 1.647011 0.015654 90)
+			(at 1.68 0.015654 90)
 			(layer "F.SilkS")
 			(effects
@@
 	)
 	(segment
-		(start 181.777447 120.626077)
-		(end 181.777447 120.027447)
-		(width 0.3)
-		(layer "F.Cu")
-		(net 13)
-	)
-	(segment
 		(start 182.100002 125.817287)
 		(end 181.85 126.067289)
@@
 	)
 	(segment
-		(start 181.777447 120.027447)
-		(end 181.75 120)
+		(start 182.237036 119.927447)
+		(end 182.209589 119.9)
 		(width 0.2)
 		(layer "F.Cu")
@@
 	)
 	(segment
+		(start 182.237036 120)
+		(end 182.237036 119.212964)
+		(width 0.8)
+		(layer "F.Cu")
+		(net 13)
+	)
+	(segment
 		(start 162.613742 98.363742)
 		(end 162.25 98)
@@
 	)
 	(segment
+		(start 182.237036 119.212964)
+		(end 182.35 119.1)
+		(width 0.8)
+		(layer "F.Cu")
+		(net 13)
+	)
+	(segment
 		(start 181.85 126.067289)
 		(end 181.85 126.796865)
@@
 	)
 	(via
-		(at 181.75 120)
-		(size 0.5)
-		(drill 0.3)
-		(layers "F.Cu" "B.Cu")
-		(net 13)
-	)
-	(via
 		(at 185.75 126.5)
 		(size 0.5)
@@
 		(net 13)
 	)
+	(via
+		(at 182.35 119.1)
+		(size 0.4)
+		(drill 0.2)
+		(layers "F.Cu" "B.Cu")
+		(net 13)
+	)
 	(segment
 		(start 157.475 101.399998)
@@
 	)
 	(segment
-		(start 182.100002 121.661355)
-		(end 182.734346 121.027011)
+		(start 182.349287 121.591)
+		(end 182.798589 121.591)
 		(width 0.2)
 		(layer "F.Cu")
@@
 	(segment
 		(start 182.100002 122.565285)
-		(end 182.100002 121.661355)
+		(end 182.100002 121.840285)
 		(width 0.2)
 		(layer "F.Cu")
@@
 	)
 	(segment
-		(start 182.734346 121.027011)
-		(end 183.15073 120.610627)
+		(start 182.100002 121.840285)
+		(end 182.349287 121.591)
 		(width 0.2)
 		(layer "F.Cu")
@@
 	)
 	(segment
-		(start 183.15073 120.610627)
-		(end 183.673554 120.610627)
+		(start 182.798589 121.591)
+		(end 184.409589 119.98)
 		(width 0.2)
 		(layer "F.Cu")
@@
 	)
 	(segment
-		(start 180.038651 120.066412)
-		(end 180.428191 120.066412)
+		(start 181.15 120)
+		(end 180.078651 120)
 		(width 0.2)
 		(layer "F.Cu")
@@
 	)
 	(segment
-		(start 180.428191 120.066412)
-		(end 180.990411 120.628632)
+		(start 180.078651 120)
+		(end 180.038651 120.04)
 		(width 0.2)
 		(layer "F.Cu")
@@
 	)
 	(segment
-		(start 180.75 123.8)
-		(end 181.109715 123.8)
+		(start 180.038651 123.088651)
+		(end 180.038651 121.026412)
 		(width 0.2)
 		(layer "F.Cu")
@@
 	)
 	(segment
-		(start 180.038651 121.026412)
-		(end 180.038651 123.088651)
+		(start 181.45 124.140285)
+		(end 181.109715 123.8)
 		(width 0.2)
 		(layer "F.Cu")
@@
 	)
 	(segment
-		(start 181.109715 123.8)
-		(end 181.45 124.140285)
+		(start 180.75 123.8)
+		(end 180.038651 123.088651)
 		(width 0.2)
 		(layer "F.Cu")
@@
 	)
 	(segment
-		(start 180.038651 123.088651)
+		(start 181.109715 123.8)
 		(end 180.75 123.8)
 		(width 0.2)
@@
 	)
 	(segment
-		(start 180.038651 121.026412)
-		(end 178.526412 121.026412)
+		(start 178.5 121)
+		(end 177.75 120.25)
 		(width 0.2)
 		(layer "F.Cu")
@@
 	)
 	(segment
-		(start 178.526412 121.026412)
-		(end 177.75 120.25)
+		(start 181.45 124.865285)
+		(end 181.45 124.140285)
 		(width 0.2)
 		(layer "F.Cu")
@@
 	)
 	(segment
-		(start 181.45 124.140285)
-		(end 181.45 124.865285)
+		(start 180.038651 121)
+		(end 178.5 121)
 		(width 0.2)
 		(layer "F.Cu")
@@
 	)
 	(segment
-		(start 182.75 124.865285)
-		(end 183.673554 123.941731)
+		(start 184.409589 123.205696)
+		(end 184.409589 121)
 		(width 0.2)
 		(layer "F.Cu")
@@
 	)
 	(segment
-		(start 183.673554 123.941731)
-		(end 183.673554 121.111627)
+		(start 182.75 124.865285)
+		(end 184.409589 123.205696)
 		(width 0.2)
 		(layer "F.Cu")
@@
 	)
 	(segment
-		(start 181.45 122.565285)
-		(end 181.45 121.604524)
+		(start 181.45 121.807036)
+		(end 182.237036 121.02)
 		(width 0.2)
 		(layer "F.Cu")
@@
 	)
 	(segment
-		(start 181.45 121.604524)
-		(end 181.777447 121.277077)
+		(start 181.45 122.565285)
+		(end 181.45 121.807036)
 		(width 0.2)
 		(layer "F.Cu")
@@
 	)
 	(segment
-		(start 180.990411 121.128632)
-		(end 180.800002 121.319041)
+		(start 180.800002 122.565285)
+		(end 180.800002 121.369998)
 		(width 0.2)
 		(layer "F.Cu")
@@
 	)
 	(segment
-		(start 180.800002 121.319041)
-		(end 180.800002 122.565285)
+		(start 180.800002 121.369998)
+		(end 181.15 121.02)
 		(width 0.2)
 		(layer "F.Cu")

Commit message: resizing
Parts:
- moved C26 0.92 mm to (187.9, 104.4)
- moved C29 0.81 mm to (189.2, 103.9)
- moved J2 0.55 mm to (180.5, 83.3)
- moved R16 0.53 mm to (170.2, 112.5)
- moved R14 0.50 mm to (190.4, 114.2)
- moved R10 0.35 mm to (186.1, 112.5)
- moved R9 0.35 mm to (186.1, 114.5)
- moved C19 0.31 mm to (171.3, 115.4)
- moved R17 0.23 mm to (159.7, 114.3)
Routing:
- net +3.3V: track 60.7 -> 62.5 mm, vias 14 -> 15
- net GNDREF: track 5.33 -> 3.81 mm, vias 35 -> 33
- net unconnected-(IC2-PC9-Pad40): track 1.01 -> 0.00 mm
- net Net-(J6-CC1): track 2.54 -> 2.04 mm

Commit message: resizing
Parts:
- L1, L2: footprint Inductor_SMD:L_2010_5025Metric -> drone_footprints:IND_FXL0530_CMT
- moved R8 4.45 mm to (156.4, 110.8), turned to -90 degrees
- moved R6 4.45 mm to (155.3, 110.8), turned to -90 degrees
- moved R7 4.44 mm to (157.6, 110.8), turned to 90 degrees
- moved R19 1.65 mm to (173.4, 123.2)
- moved R20 1.65 mm to (173.3, 124.3)
- moved R21 1.65 mm to (173.3, 125.4)
- moved C30 1.60 mm to (168.8, 118.6)
- moved C8 1.60 mm to (166.2, 119.3)
- moved C9 1.60 mm to (166.2, 122.5)
- moved Q1 1.60 mm to (168.9, 121.9)
- moved L1 1.43 mm to (158.1, 106.7)
- moved C10 0.86 mm to (184.2, 120.7)
- moved C12 0.86 mm to (180.9, 120.7)
- moved R1 0.86 mm to (185.3, 120.6)
- moved R18 0.86 mm to (182.0, 120.6)
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Routing:
- net +5VBAT: track 8.88 -> 14.0 mm
- net Net-(U4-FB): track 10.3 -> 15.0 mm
- net Net-(U2-FB): track 10.0 -> 12.9 mm
- net Net-(U4-SW): track 7.23 -> 9.31 mm
- net Net-(U2-SW): track 8.20 -> 9.63 mm
- net /GPS_TX: track 26.6 -> 27.4 mm
- net /GPS_RX: track 25.7 -> 26.4 mm
